File: 32X_main1.kicad_sch (KiCad schematic)
At the start: 27 parts, among them IC504 315-5818, IC505 315-5805, IC509 74AC04

Commit message: Ferrite Bead LCSC Part update
Parts:
- FB7: LCSC Part # (none) -> C41330
- FB7: LCSC Part # (none) -> C124102
Changed lines of the file:
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@@
       (effects (font (size 1.27 1.27)) hide)
     )
-    (property "LCSC Part #" "" (at 263.525 203.2 0)
+    (property "LCSC Part #" "C41330" (at 263.525 203.2 0)
       (effects (font (size 1.27 1.27)) hide)
     )
@@
       (effects (font (size 1.27 1.27)) hide)
     )
-    (property "LCSC Part #" "" (at 153.67 179.705 0)
+    (property "LCSC Part #" "C124102" (at 153.67 179.705 0)
       (effects (font (size 1.27 1.27)) hide)
     )
@@
       (effects (font (size 1.27 1.27)) hide)
     )
-    (property "LCSC Part #" "" (at 132.715 156.845 0)
-      (effects (font (size 1.27 1.27)) hide)
-    )
+    (property "LCSC Part #" "C41330" (at 132.715 156.845 0)
+      (effects (font (size 1.27 1.27)) hide)
+    )

Commit message: Added more JLC Part numbers
Parts:
- IC509: LCSC Part # (none) -> C352940
- L501: LCSC Part # (none) -> C27775
Changed lines of the file:
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@@
       (effects (font (size 1.27 1.27)) hide)
     )
-    (property "LCSC Part #" "" (at 77.47 247.65 0)
+    (property "LCSC Part #" "C352940" (at 77.47 247.65 0)
       (effects (font (size 1.27 1.27)) hide)
     )
@@
       (effects (font (size 1.27 1.27)) hide)
     )
-    (property "LCSC Part #" "" (at 278.13 244.475 0)
+    (property "LCSC Part #" "C352940" (at 278.13 244.475 0)
       (effects (font (size 1.27 1.27)) hide)
     )
@@
       (effects (font (size 1.27 1.27)) hide)
     )
-    (property "LCSC Part #" "" (at 98.425 247.65 0)
+    (property "LCSC Part #" "C352940" (at 98.425 247.65 0)
       (effects (font (size 1.27 1.27)) hide)
     )
@@
       (effects (font (size 1.27 1.27)) hide)
     )
-    (property "LCSC Part #" "" (at 118.11 156.845 0)
+    (property "LCSC Part #" "C352940" (at 118.11 156.845 0)
       (effects (font (size 1.27 1.27)) hide)
     )
@@
       (effects (font (size 1.27 1.27)) hide)
     )
-    (property "LCSC Part #" "" (at 203.835 170.815 0)
+    (property "LCSC Part #" "C27775" (at 203.835 170.815 0)
       (effects (font (size 1.27 1.27)) hide)
     )
@@
       (effects (font (size 1.27 1.27)) hide)
     )
-    (property "LCSC Part #" "" (at 249.555 203.2 0)
-      (effects (font (size 1.27 1.27)) hide)
-    )
+    (property "LCSC Part #" "C352940" (at 249.555 203.2 0)
+      (effects (font (size 1.27 1.27)) hide)
+    )

Commit message: more component parts updated
Full in the * as PAL versions.
Added MPN for PCBWAY
Parts:
- C5: MPN (none) -> VJ0805Y104JXJMT
- C5: MPN (none) -> VJ1206V475MXJTW1BC
- FB7: MPN (none) -> CBG201209U121T
- FB7: MPN (none) -> CBG201209U000T
- FB7: MPN (none) -> CBG201209U221T
- IC509: MPN (none) -> SN74AC04DR
- L501: MPN (none) -> CMI322513J101KT
- R561: MPN (none) -> CRCW08058K20FKEA
- R562: MPN (none) -> CRCW08052K00JNEA
- R566: MPN (none) -> CRCW08054K70JNEAC
- RM3, RM4, RM5, RM6: MPN (none) -> YC164-FR-0710KL
Changed lines of the file:
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@@
+      (effects (font (size 1.27 1.27)) hide)
+    )
+    (property "MPN" "CRCW08054K70JNEAC" (at 49.53 125.73 0)
       (effects (font (size 1.27 1.27)) hide)
     )
@@
     )
     (property "LCSC Part #" "C352940" (at 77.47 247.65 0)
+      (effects (font (size 1.27 1.27)) hide)
+    )
+    (property "MPN" "SN74AC04DR" (at 77.47 247.65 0)
       (effects (font (size 1.27 1.27)) hide)
     )
@@
       (effects (font (size 1.27 1.27)) hide)
     )
+    (property "MPN" "VJ0805Y104JXJMT" (at 195.58 243.84 0)
+      (effects (font (size 1.27 1.27)) hide)
+    )
     (pin "1")
     (pin "2")
@@
     )
     (property "LCSC Part #" "C352940" (at 278.13 244.475 0)
+      (effects (font (size 1.27 1.27)) hide)
+    )
+    (property "MPN" "SN74AC04DR" (at 278.13 244.475 0)
       (effects (font (size 1.27 1.27)) hide)
     )
@@
       (effects (font (size 1.27 1.27)) hide)
     )
+    (property "MPN" "VJ0805Y104JXJMT" (at 194.945 183.515 0)
+      (effects (font (size 1.27 1.27)) hide)
+    )
     (pin "1")
     (pin "2")
@@
     )
     (property "LCSC Part #" "C110924" (at 85.725 65.405 0)
+      (effects (font (size 1.27 1.27)) hide)
+    )
+    (property "MPN" "YC164-FR-0710KL" (at 85.725 65.405 0)
       (effects (font (size 1.27 1.27)) hide)
     )
@@
       (effects (font (size 1.27 1.27)) hide)
     )
+    (property "MPN" "VJ1206V475MXJTW1BC" (at 207.645 243.84 0)
+      (effects (font (size 1.27 1.27)) hide)
+    )
     (pin "1")
     (pin "2")
@@
       (effects (font (size 1.27 1.27)) hide)
     )
+    (property "MPN" "VJ1206V475MXJTW1BC" (at 291.465 161.29 0)
+      (effects (font (size 1.27 1.27)) hide)
+    )
     (pin "1")
     (pin "2")
@@
       (effects (font (size 1.27 1.27)) hide)
     )
+    (property "MPN" "VJ0805Y104JXJMT" (at 272.415 161.29 0)
+      (effects (font (size 1.27 1.27)) hide)
+    )
     (pin "1")
     (pin "2")
@@
       (effects (font (size 1.27 1.27)) hide)
     )
+    (property "MPN" "VJ0805Y104JXJMT" (at 282.575 161.29 0)
+      (effects (font (size 1.27 1.27)) hide)
+    )
     (pin "1")
     (pin "2")
@@
       (effects (font (size 1.27 1.27)) hide)
     )
+    (property "MPN" "" (at 108.585 198.755 0)
+      (effects (font (size 1.27 1.27)) hide)
+    )
     (pin "1")
     (pin "2")
@@
       (effects (font (size 1.27 1.27)) hide)
     )
+    (property "MPN" "CBG201209U121T" (at 263.525 203.2 0)
+      (effects (font (size 1.27 1.27)) hide)
+    )
     (pin "1")
     (pin "2")
@@
       (effects (font (size 1.27 1.27)) hide)
     )
+    (property "MPN" "" (at 118.11 184.785 0)
+      (effects (font (size 1.27 1.27)) hide)
+    )
     (pin "1")
     (pin "2")
@@
       (effects (font (size 1.27 1.27)) hide)
     )
+    (property "MPN" "" (at 232.41 243.84 0)
+      (effects (font (size 1.27 1.27)) hide)
+    )
     (pin "1")
     (pin "2")
@@
       (effects (font (size 1.27 1.27)) hide)
     )
+    (property "MPN" "CBG201209U000T" (at 236.22 203.2 0)
+      (effects (font (size 1.27 1.27)) hide)
+    )
     (pin "1")
     (pin "2")
@@
       (effects (font (size 1.27 1.27)) hide)
     )
+    (property "MPN" "CBG201209U000T" (at 153.67 169.545 0)
+      (effects (font (size 1.27 1.27)) hide)
+    )
     (pin "1")
     (pin "2")
@@
     )
     (property "LCSC Part #" "C352940" (at 98.425 247.65 0)
+      (effects (font (size 1.27 1.27)) hide)
+    )
+    (property "MPN" "SN74AC04DR" (at 98.425 247.65 0)
       (effects (font (size 1.27 1.27)) hide)
     )
@@
       (effects (font (size 1.27 1.27)) hide)
     )
+    (property "MPN" "YC164-FR-0710KL" (at 85.725 104.14 0)
+      (effects (font (size 1.27 1.27)) hide)
+    )
     (pin "1")
     (pin "2")
@@
     )
     (property "LCSC Part #" "C352940" (at 118.11 156.845 0)
+      (effects (font (size 1.27 1.27)) hide)
+    )
+    (property "MPN" "SN74AC04DR" (at 118.11 156.845 0)
       (effects (font (size 1.27 1.27)) hide)
     )
@@
       (effects (font (size 1.27 1.27)) hide)
     )
+    (property "MPN" "CRCW08058K20FKEA" (at 88.265 234.315 0)
+      (effects (font (size 1.27 1.27)) hide)
+    )
     (pin "1")
     (pin "2")
@@
     )
     (property "LCSC Part #" "C110924" (at 85.725 84.455 0)
+      (effects (font (size 1.27 1.27)) hide)
+    )
+    (property "MPN" "YC164-FR-0710KL" (at 85.725 84.455 0)
       (effects (font (size 1.27 1.27)) hide)
     )
@@
       (effects (font (size 1.27 1.27)) hide)
     )
+    (property "MPN" "CRCW08052K00JNEA" (at 59.055 247.65 0)
+      (effects (font (size 1.27 1.27)) hide)
+    )
     (pin "1")
     (pin "2")
@@
       (effects (font (size 1.27 1.27)) hide)
     )
+    (property "MPN" "CMI322513J101KT" (at 203.835 170.815 0)
+      (effects (font (size 1.27 1.27)) hide)
+    )
     (pin "1")
     (pin "2")
@@
     )
     (property "LCSC Part #" "C2182015" (at 220.345 243.84 0)
+      (effects (font (size 1.27 1.27)) hide)
+    )
+    (property "MPN" "VJ1206V475MXJTW1BC" (at 220.345 243.84 0)
       (effects (font (size 1.27 1.27)) hide)
     )
@@
     )
     (property "LCSC Part #" "" (at 249.555 48.26 0)
+      (effects (font (size 1.27 1.27)) hide)
+    )
+    (property "MPN" "" (at 249.555 48.26 0)
       (effects (font (size 1.27 1.27)) hide)
     )
@@
       (effects (font (size 1.27 1.27)) hide)
     )
+    (property "MPN" "VJ1206V475MXJTW1BC" (at 203.835 183.515 0)
+      (effects (font (size 1.27 1.27)) hide)
+    )
     (pin "1")
     (pin "2")
@@
     )
     (property "LCSC Part #" "C352940" (at 249.555 203.2 0)
+      (effects (font (size 1.27 1.27)) hide)
+    )
+    (property "MPN" "SN74AC04DR" (at 249.555 203.2 0)
       (effects (font (size 1.27 1.27)) hide)
     )
@@
       (effects (font (size 1.27 1.27)) hide)
     )
+    (property "MPN" "CBG201209U221T" (at 153.67 179.705 0)
+      (effects (font (size 1.27 1.27)) hide)
+    )
     (pin "1")
     (pin "2")
@@
       (effects (font (size 1.27 1.27)) hide)
     )
+    (property "MPN" "CBG201209U121T" (at 132.715 156.845 0)
+      (effects (font (size 1.27 1.27)) hide)
+    )
     (pin "1")
     (pin "2")
@@
     )
     (property "LCSC Part #" "C110924" (at 85.725 123.19 0)
+      (effects (font (size 1.27 1.27)) hide)
+    )
+    (property "MPN" "YC164-FR-0710KL" (at 85.725 123.19 0)
       (effects (font (size 1.27 1.27)) hide)
     )
@@
       (effects (font (size 1.27 1.27)) hide)
     )
+    (property "MPN" "" (at 176.53 48.26 0)
+      (effects (font (size 1.27 1.27)) hide)
+    )

Commit message: Allow for both wide and narrow IC509.
Parts:
- IC509: footprint Package_SO:SO-14_5.3x10.2mm_P1.27mm -> Neptune:SO-14_Dual_Purpose_P1.27mm
Changed lines of the file:
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@@
       (effects (font (size 1.27 1.27)))
     )
-    (property "Footprint" "Package_SO:SO-14_5.3x10.2mm_P1.27mm" (at 77.47 247.65 0)
+    (property "Footprint" "Neptune:SO-14_Dual_Purpose_P1.27mm" (at 77.47 247.65 0)
       (effects (font (size 1.27 1.27)) hide)
     )
@@
       (effects (font (size 1.27 1.27)) (justify left))
     )
-    (property "Footprint" "Package_SO:SO-14_5.3x10.2mm_P1.27mm" (at 278.13 244.475 0)
+    (property "Footprint" "Neptune:SO-14_Dual_Purpose_P1.27mm" (at 278.13 244.475 0)
       (effects (font (size 1.27 1.27)) hide)
     )
@@
       (effects (font (size 1.27 1.27)))
     )
-    (property "Footprint" "Package_SO:SO-14_5.3x10.2mm_P1.27mm" (at 98.425 247.65 0)
+    (property "Footprint" "Neptune:SO-14_Dual_Purpose_P1.27mm" (at 98.425 247.65 0)
       (effects (font (size 1.27 1.27)) hide)
     )
@@
       (effects (font (size 1.27 1.27)))
     )
-    (property "Footprint" "Package_SO:SO-14_5.3x10.2mm_P1.27mm" (at 118.11 156.845 0)
+    (property "Footprint" "Neptune:SO-14_Dual_Purpose_P1.27mm" (at 118.11 156.845 0)
       (effects (font (size 1.27 1.27)) hide)
     )
@@
       (effects (font (size 1.27 1.27)))
     )
-    (property "Footprint" "Package_SO:SO-14_5.3x10.2mm_P1.27mm" (at 249.555 203.2 0)
-      (effects (font (size 1.27 1.27)) hide)
-    )
+    (property "Footprint" "Neptune:SO-14_Dual_Purpose_P1.27mm" (at 249.555 203.2 0)
+      (effects (font (size 1.27 1.27)) hide)
+    )

Commit message: Update LCSC parts
Parts:
- C5: LCSC Part # C2237864 -> C111492
- C5: LCSC Part # C2182015 -> C132170
- R562: LCSC Part # C2077049 -> C114231
Changed lines of the file:
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@@
       (effects (font (size 1.27 1.27)) hide)
     )
-    (property "LCSC Part #" "C2237864" (at 195.58 243.84 0)
+    (property "LCSC Part #" "C111492" (at 195.58 243.84 0)
       (effects (font (size 1.27 1.27)) hide)
     )
@@
       (effects (font (size 1.27 1.27)) hide)
     )
-    (property "LCSC Part #" "C2237864" (at 194.945 183.515 0)
+    (property "LCSC Part #" "C111492" (at 194.945 183.515 0)
       (effects (font (size 1.27 1.27)) hide)
     )
@@
       (effects (font (size 1.27 1.27)) hide)
     )
-    (property "LCSC Part #" "C2182015" (at 207.645 243.84 0)
+    (property "LCSC Part #" "C132170" (at 207.645 243.84 0)
       (effects (font (size 1.27 1.27)) hide)
     )
@@
       (effects (font (size 1.27 1.27)) hide)
     )
-    (property "LCSC Part #" "C2182015" (at 291.465 161.29 0)
+    (property "LCSC Part #" "C132170" (at 291.465 161.29 0)
       (effects (font (size 1.27 1.27)) hide)
     )
@@
       (effects (font (size 1.27 1.27)) hide)
     )
-    (property "LCSC Part #" "C2237864" (at 272.415 161.29 0)
+    (property "LCSC Part #" "C111492" (at 272.415 161.29 0)
       (effects (font (size 1.27 1.27)) hide)
     )
@@
       (effects (font (size 1.27 1.27)) hide)
     )
-    (property "LCSC Part #" "C2237864" (at 282.575 161.29 0)
+    (property "LCSC Part #" "C111492" (at 282.575 161.29 0)
       (effects (font (size 1.27 1.27)) hide)
     )
@@
       (effects (font (size 1.27 1.27)) hide)
     )
-    (property "LCSC Part #" "C2077049" (at 59.055 247.65 0)
+    (property "LCSC Part #" "C114231" (at 59.055 247.65 0)
       (effects (font (size 1.27 1.27)) hide)
     )
@@
       (effects (font (size 1.27 1.27)) hide)
     )
-    (property "LCSC Part #" "C2182015" (at 220.345 243.84 0)
+    (property "LCSC Part #" "C132170" (at 220.345 243.84 0)
       (effects (font (size 1.27 1.27)) hide)
     )
@@
       (effects (font (size 1.27 1.27)) hide)
     )
-    (property "LCSC Part #" "C2182015" (at 203.835 183.515 0)
-      (effects (font (size 1.27 1.27)) hide)
-    )
+    (property "LCSC Part #" "C132170" (at 203.835 183.515 0)
+      (effects (font (size 1.27 1.27)) hide)
+    )

Commit message: Longer pads for IC505.
Parts:
- IC505: footprint Package_QFP:PQFP-80_14x20mm_P0.8mm -> Neptune:PQFP-80_14x20mm_P0.8mm
Changed lines of the file:
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@@
       (effects (font (size 1.27 1.27)))
     )
-    (property "Footprint" "Package_QFP:PQFP-80_14x20mm_P0.8mm" (at 249.555 83.82 0)
+    (property "Footprint" "Neptune:PQFP-80_14x20mm_P0.8mm" (at 249.555 83.82 0)
       (effects (font (size 1.27 1.27)) hide)
     )
