File: sge.kicad_sch (KiCad schematic)
At the start: 27 parts, among them IC6 315-5660

Commit message: Added resistor array parts
Parts:
- RA608: LCSC Part # (none) -> C136829; MPN (none) -> YC164-JR-072K2L
Changed lines of the file:
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@@
+      (effects (font (size 1.27 1.27)) hide)
+    )
+    (property "LCSC Part #" "C136829" (at 127 258.445 0)
+      (effects (font (size 1.27 1.27)) hide)
+    )
+    (property "MPN" "YC164-JR-072K2L" (at 127 258.445 0)
       (effects (font (size 1.27 1.27)) hide)
     )

Commit message: Update LCSC parts
Parts:
- C1: LCSC Part # C2224419 -> C520037
- C1: LCSC Part # C2237538 -> C149613
- C2: LCSC Part # C2232461 -> C520060
- C8: LCSC Part # C1850591 -> C541528
- R3: LCSC Part # C3008897 -> C114561
- R3: LCSC Part # C313845 -> C136926
- RA1, RA2, RA3, RA4, RA5: LCSC Part # C136838 -> C1852225
Changed lines of the file:
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@@
       (effects (font (size 1.27 1.27)) hide)
     )
-    (property "LCSC Part #" "C136838" (at 113.03 38.1 0)
+    (property "LCSC Part #" "C1852225" (at 113.03 38.1 0)
       (effects (font (size 1.27 1.27)) hide)
     )
@@
       (effects (font (size 1.27 1.27)) hide)
     )
-    (property "LCSC Part #" "C3008897" (at 139.7 258.445 0)
+    (property "LCSC Part #" "C114561" (at 139.7 258.445 0)
       (effects (font (size 1.27 1.27)) hide)
     )
@@
       (effects (font (size 1.27 1.27)) hide)
     )
-    (property "LCSC Part #" "C136838" (at 99.06 38.1 0)
+    (property "LCSC Part #" "C1852225" (at 99.06 38.1 0)
       (effects (font (size 1.27 1.27)) hide)
     )
@@
       (effects (font (size 1.27 1.27)) hide)
     )
-    (property "LCSC Part #" "C136838" (at 124.46 38.1 0)
+    (property "LCSC Part #" "C1852225" (at 124.46 38.1 0)
       (effects (font (size 1.27 1.27)) hide)
     )
@@
       (effects (font (size 1.27 1.27)) hide)
     )
-    (property "LCSC Part #" "C136838" (at 116.84 38.1 0)
+    (property "LCSC Part #" "C1852225" (at 116.84 38.1 0)
       (effects (font (size 1.27 1.27)) hide)
     )
@@
       (effects (font (size 1.27 1.27)) hide)
     )
-    (property "LCSC Part #" "C136838" (at 198.12 38.1 0)
+    (property "LCSC Part #" "C1852225" (at 198.12 38.1 0)
       (effects (font (size 1.27 1.27)) hide)
     )
@@
       (effects (font (size 1.27 1.27)) hide)
     )
-    (property "LCSC Part #" "C2232461" (at 261.62 260.985 0)
+    (property "LCSC Part #" "C520060" (at 261.62 260.985 0)
       (effects (font (size 1.27 1.27)) hide)
     )
@@
       (effects (font (size 1.27 1.27)) hide)
     )
-    (property "LCSC Part #" "C3008897" (at 392.43 52.07 0)
+    (property "LCSC Part #" "C114561" (at 392.43 52.07 0)
       (effects (font (size 1.27 1.27)) hide)
     )
@@
       (effects (font (size 1.27 1.27)) hide)
     )
-    (property "LCSC Part #" "C2224419" (at 175.26 264.16 0)
+    (property "LCSC Part #" "C520037" (at 175.26 264.16 0)
       (effects (font (size 1.27 1.27)) hide)
     )
@@
       (effects (font (size 1.27 1.27)) hide)
     )
-    (property "LCSC Part #" "C1850591" (at 30.48 174.625 0)
+    (property "LCSC Part #" "C541528" (at 30.48 174.625 0)
       (effects (font (size 1.27 1.27)) hide)
     )
@@
       (effects (font (size 1.27 1.27)) hide)
     )
-    (property "LCSC Part #" "C2224419" (at 160.655 264.16 0)
+    (property "LCSC Part #" "C520037" (at 160.655 264.16 0)
       (effects (font (size 1.27 1.27)) hide)
     )
@@
       (effects (font (size 1.27 1.27)) hide)
     )
-    (property "LCSC Part #" "C2224419" (at 295.275 238.125 0)
+    (property "LCSC Part #" "C520037" (at 295.275 238.125 0)
       (effects (font (size 1.27 1.27)) hide)
     )
@@
       (effects (font (size 1.27 1.27)) hide)
     )
-    (property "LCSC Part #" "C136838" (at 135.89 38.1 0)
+    (property "LCSC Part #" "C1852225" (at 135.89 38.1 0)
       (effects (font (size 1.27 1.27)) hide)
     )
@@
       (effects (font (size 1.27 1.27)) hide)
     )
-    (property "LCSC Part #" "C136838" (at 120.65 38.1 0)
+    (property "LCSC Part #" "C1852225" (at 120.65 38.1 0)
       (effects (font (size 1.27 1.27)) hide)
     )
@@
       (effects (font (size 1.27 1.27)) hide)
     )
-    (property "LCSC Part #" "C136838" (at 179.07 38.1 0)
+    (property "LCSC Part #" "C1852225" (at 179.07 38.1 0)
       (effects (font (size 1.27 1.27)) hide)
     )
@@
       (effects (font (size 1.27 1.27)) hide)
     )
-    (property "LCSC Part #" "C3008897" (at 354.33 229.87 0)
+    (property "LCSC Part #" "C114561" (at 354.33 229.87 0)
       (effects (font (size 1.27 1.27)) hide)
     )
@@
       (effects (font (size 1.27 1.27)) hide)
     )
-    (property "LCSC Part #" "C136838" (at 132.08 38.1 0)
+    (property "LCSC Part #" "C1852225" (at 132.08 38.1 0)
       (effects (font (size 1.27 1.27)) hide)
     )
@@
       (effects (font (size 1.27 1.27)) hide)
     )
-    (property "LCSC Part #" "C136838" (at 201.93 38.1 0)
+    (property "LCSC Part #" "C1852225" (at 201.93 38.1 0)
       (effects (font (size 1.27 1.27)) hide)
     )
@@
       (effects (font (size 1.27 1.27)) hide)
     )
-    (property "LCSC Part #" "C2224419" (at 321.31 238.125 0)
+    (property "LCSC Part #" "C520037" (at 321.31 238.125 0)
       (effects (font (size 1.27 1.27)) hide)
     )
@@
       (effects (font (size 1.27 1.27)) hide)
     )
-    (property "LCSC Part #" "C136838" (at 194.31 38.1 0)
+    (property "LCSC Part #" "C1852225" (at 194.31 38.1 0)
       (effects (font (size 1.27 1.27)) hide)
     )
@@
       (effects (font (size 1.27 1.27)) hide)
     )
-    (property "LCSC Part #" "C136838" (at 128.27 38.1 0)
+    (property "LCSC Part #" "C1852225" (at 128.27 38.1 0)
       (effects (font (size 1.27 1.27)) hide)
     )
@@
       (effects (font (size 1.27 1.27)) hide)
     )
-    (property "LCSC Part #" "C136838" (at 102.87 38.1 0)
+    (property "LCSC Part #" "C1852225" (at 102.87 38.1 0)
       (effects (font (size 1.27 1.27)) hide)
     )
@@
       (effects (font (size 1.27 1.27)) hide)
     )
-    (property "LCSC Part #" "C2224419" (at 314.96 238.125 0)
+    (property "LCSC Part #" "C520037" (at 314.96 238.125 0)
       (effects (font (size 1.27 1.27)) hide)
     )
@@
       (effects (font (size 1.27 1.27)) hide)
     )
-    (property "LCSC Part #" "C136838" (at 80.01 38.1 0)
+    (property "LCSC Part #" "C1852225" (at 80.01 38.1 0)
       (effects (font (size 1.27 1.27)) hide)
     )
@@
       (effects (font (size 1.27 1.27)) hide)
     )
-    (property "LCSC Part #" "C136838" (at 190.5 38.1 0)
+    (property "LCSC Part #" "C1852225" (at 190.5 38.1 0)
       (effects (font (size 1.27 1.27)) hide)
     )
@@
       (effects (font (size 1.27 1.27)) hide)
     )
-    (property "LCSC Part #" "C136838" (at 139.7 38.1 0)
+    (property "LCSC Part #" "C1852225" (at 139.7 38.1 0)
       (effects (font (size 1.27 1.27)) hide)
     )
@@
       (effects (font (size 1.27 1.27)) hide)
     )
-    (property "LCSC Part #" "C313845" (at 234.95 247.65 0)
+    (property "LCSC Part #" "C136926" (at 234.95 247.65 0)
       (effects (font (size 1.27 1.27)) hide)
     )
@@
       (effects (font (size 1.27 1.27)) hide)
     )
-    (property "LCSC Part #" "C136838" (at 205.74 38.1 0)
+    (property "LCSC Part #" "C1852225" (at 205.74 38.1 0)
       (effects (font (size 1.27 1.27)) hide)
     )
@@
       (effects (font (size 1.27 1.27)) hide)
     )
-    (property "LCSC Part #" "C2237538" (at 388.62 72.39 0)
+    (property "LCSC Part #" "C149613" (at 388.62 72.39 0)
       (effects (font (size 1.27 1.27)) hide)
     )
@@
       (effects (font (size 1.27 1.27)) hide)
     )
-    (property "LCSC Part #" "C136838" (at 95.25 38.1 0)
+    (property "LCSC Part #" "C1852225" (at 95.25 38.1 0)
       (effects (font (size 1.27 1.27)) hide)
     )
@@
       (effects (font (size 1.27 1.27)) hide)
     )
-    (property "LCSC Part #" "C1850591" (at 31.115 71.755 0)
+    (property "LCSC Part #" "C541528" (at 31.115 71.755 0)
       (effects (font (size 1.27 1.27)) hide)
     )
@@
       (effects (font (size 1.27 1.27)) hide)
     )
-    (property "LCSC Part #" "C2224419" (at 200.025 264.16 0)
+    (property "LCSC Part #" "C520037" (at 200.025 264.16 0)
       (effects (font (size 1.27 1.27)) hide)
     )
@@
       (effects (font (size 1.27 1.27)) hide)
     )
-    (property "LCSC Part #" "C136838" (at 186.69 38.1 0)
+    (property "LCSC Part #" "C1852225" (at 186.69 38.1 0)
       (effects (font (size 1.27 1.27)) hide)
     )
@@
       (effects (font (size 1.27 1.27)) hide)
     )
-    (property "LCSC Part #" "C2224419" (at 187.96 264.16 0)
+    (property "LCSC Part #" "C520037" (at 187.96 264.16 0)
       (effects (font (size 1.27 1.27)) hide)
     )
@@
       (effects (font (size 1.27 1.27)) hide)
     )
-    (property "LCSC Part #" "C136838" (at 182.88 38.1 0)
-      (effects (font (size 1.27 1.27)) hide)
-    )
+    (property "LCSC Part #" "C1852225" (at 182.88 38.1 0)
+      (effects (font (size 1.27 1.27)) hide)
+    )

Commit message: BOM tweaks.
Parts:
- C1: value 47pF -> 47pF (PAL only)
- C2: value 33pF -> 33pF (PAL only)
- RA1, RA2, RA3, RA4, RA5: value R_Pack04_Split -> 4x100
- RA6: value R_Pack02_Split -> 2x100
Other:
- note removed: "PAL ONLY"
Changed lines of the file:
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@@
     (title "SGE (MD Custom ASIC)")
     (date "2023-11-29")
-    (rev "1.1b")
+    (rev "1.2a")
     (company "By Cosam")
     (comment 1 "Neptune")
@@
     (stroke (width 0) (type default))
   )
-  (text "PAL\nONLY" (at 398.145 74.295 0)
-    (effects (font (size 1.27 1.27)) (justify left bottom))
-  )
   (text "Using 32X's RESET means we\ndon't need the whole /MRES\nto /SRES circuit from the MD."
     (at 15.875 61.595 0)
@@
     (effects (font (size 1.27 1.27)) (justify left bottom))
   )
-  (text "PAL\nONLY" (at 271.145 262.89 0)
-    (effects (font (size 1.27 1.27)) (justify left bottom))
-  )
   (label "ZD7" (at 367.665 114.3 0) (fields_autoplaced)
     (effects (font (size 1.27 1.27)) (justify left bottom))
@@
       (effects (font (size 1.27 1.27)) (justify left))
     )
-    (property "Value" "R_Pack04_Split" (at 110.49 36.83 0)
+    (property "Value" "4x100" (at 110.49 36.83 0)
       (effects (font (size 1.27 1.27)) (justify left) hide)
     )
@@
       (effects (font (size 1.27 1.27)) (justify left))
     )
-    (property "Value" "R_Pack04_Split" (at 101.6 36.83 0)
+    (property "Value" "4x100" (at 101.6 36.83 0)
       (effects (font (size 1.27 1.27)) (justify left) hide)
     )
@@
       (effects (font (size 1.27 1.27)) (justify left))
     )
-    (property "Value" "R_Pack04_Split" (at 121.92 36.83 0)
+    (property "Value" "4x100" (at 121.92 36.83 0)
       (effects (font (size 1.27 1.27)) (justify left) hide)
     )
@@
       (effects (font (size 1.27 1.27)) (justify left))
     )
-    (property "Value" "R_Pack04_Split" (at 114.3 36.83 0)
+    (property "Value" "4x100" (at 114.3 36.83 0)
       (effects (font (size 1.27 1.27)) (justify left) hide)
     )
@@
       (effects (font (size 1.27 1.27)) (justify left))
     )
-    (property "Value" "R_Pack04_Split" (at 200.66 36.83 0)
+    (property "Value" "4x100" (at 200.66 36.83 0)
       (effects (font (size 1.27 1.27)) (justify left) hide)
     )
@@
       (effects (font (size 1.27 1.27)) (justify left))
     )
-    (property "Value" "33pF" (at 265.43 262.255 0)
+    (property "Value" "33pF (PAL only)" (at 265.43 262.255 0)
       (effects (font (size 1.27 1.27)) (justify left))
     )
@@
       (effects (font (size 1.27 1.27)) (justify left))
     )
-    (property "Value" "R_Pack02_Split" (at 109.22 36.83 0)
+    (property "Value" "2x100" (at 109.22 36.83 0)
       (effects (font (size 1.27 1.27)) (justify left) hide)
     )
@@
       (effects (font (size 1.27 1.27)) (justify left))
     )
-    (property "Value" "R_Pack04_Split" (at 138.43 36.83 0)
+    (property "Value" "4x100" (at 138.43 36.83 0)
       (effects (font (size 1.27 1.27)) (justify left) hide)
     )
@@
       (effects (font (size 1.27 1.27)) (justify left))
     )
-    (property "Value" "R_Pack02_Split" (at 86.36 36.83 0)
+    (property "Value" "2x100" (at 86.36 36.83 0)
       (effects (font (size 1.27 1.27)) (justify left) hide)
     )
@@
       (effects (font (size 1.27 1.27)) (justify left))
     )
-    (property "Value" "R_Pack04_Split" (at 118.11 36.83 0)
+    (property "Value" "4x100" (at 118.11 36.83 0)
       (effects (font (size 1.27 1.27)) (justify left) hide)
     )
@@
       (effects (font (size 1.27 1.27)) (justify left))
     )
-    (property "Value" "R_Pack04_Split" (at 176.53 36.83 0)
+    (property "Value" "4x100" (at 176.53 36.83 0)
       (effects (font (size 1.27 1.27)) (justify left) hide)
     )
@@
       (effects (font (size 1.27 1.27)) (justify left))
     )
-    (property "Value" "R_Pack04_Split" (at 134.62 36.83 0)
+    (property "Value" "4x100" (at 134.62 36.83 0)
       (effects (font (size 1.27 1.27)) (justify left) hide)
     )
@@
       (effects (font (size 1.27 1.27)) (justify left))
     )
-    (property "Value" "R_Pack04_Split" (at 204.47 36.83 0)
+    (property "Value" "4x100" (at 204.47 36.83 0)
       (effects (font (size 1.27 1.27)) (justify left) hide)
     )
@@
       (effects (font (size 1.27 1.27)) (justify left))
     )
-    (property "Value" "R_Pack04_Split" (at 196.85 36.83 0)
+    (property "Value" "4x100" (at 196.85 36.83 0)
       (effects (font (size 1.27 1.27)) (justify left) hide)
     )
@@
       (effects (font (size 1.27 1.27)) (justify left))
     )
-    (property "Value" "R_Pack04_Split" (at 130.81 36.83 0)
+    (property "Value" "4x100" (at 130.81 36.83 0)
       (effects (font (size 1.27 1.27)) (justify left) hide)
     )
@@
       (effects (font (size 1.27 1.27)) (justify left))
     )
-    (property "Value" "R_Pack04_Split" (at 105.41 36.83 0)
+    (property "Value" "4x100" (at 105.41 36.83 0)
       (effects (font (size 1.27 1.27)) (justify left) hide)
     )
@@
       (effects (font (size 1.27 1.27)) (justify left))
     )
-    (property "Value" "R_Pack04_Split" (at 82.55 36.83 0)
+    (property "Value" "4x100" (at 82.55 36.83 0)
       (effects (font (size 1.27 1.27)) (justify left) hide)
     )
@@
   )
   (symbol (lib_id "Device:FerriteBead_Small") (at 252.73 254.635 90) (unit 1)
-    (in_bom yes) (on_board yes) (dnp no) (fields_autoplaced)
-    (property "Reference" "FB7" (at 252.6919 250.19 90)
+    (in_bom yes) (on_board yes) (dnp no)
+    (property "Reference" "FB7" (at 252.73 251.46 90)
       (effects (font (size 1.27 1.27)))
     )
-    (property "Value" "0" (at 252.6919 250.825 90)
+    (property "Value" "0" (at 252.73 257.81 90)
       (effects (font (size 1.27 1.27)))
     )
@@
       (effects (font (size 1.27 1.27)) (justify left))
     )
-    (property "Value" "R_Pack04_Split" (at 187.96 36.83 0)
+    (property "Value" "4x100" (at 187.96 36.83 0)
       (effects (font (size 1.27 1.27)) (justify left) hide)
     )
@@
       (effects (font (size 1.27 1.27)) (justify left))
     )
-    (property "Value" "R_Pack04_Split" (at 142.24 36.83 0)
+    (property "Value" "4x100" (at 142.24 36.83 0)
       (effects (font (size 1.27 1.27)) (justify left) hide)
     )
@@
       (effects (font (size 1.27 1.27)) (justify left))
     )
-    (property "Value" "R_Pack04_Split" (at 208.28 36.83 0)
+    (property "Value" "4x100" (at 208.28 36.83 0)
       (effects (font (size 1.27 1.27)) (justify left) hide)
     )
@@
   )
   (symbol (lib_id "Device:C") (at 388.62 72.39 0) (unit 1)
-    (in_bom yes) (on_board yes) (dnp no) (fields_autoplaced)
-    (property "Reference" "C1" (at 392.43 71.12 0)
+    (in_bom yes) (on_board yes) (dnp no)
+    (property "Reference" "C1" (at 391.795 71.12 0)
       (effects (font (size 1.27 1.27)) (justify left))
     )
-    (property "Value" "47pF" (at 392.43 73.66 0)
+    (property "Value" "47pF (PAL only)" (at 391.795 73.66 0)
       (effects (font (size 1.27 1.27)) (justify left))
     )
@@
       (effects (font (size 1.27 1.27)) (justify left))
     )
-    (property "Value" "R_Pack04_Split" (at 97.79 36.83 0)
+    (property "Value" "4x100" (at 97.79 36.83 0)
       (effects (font (size 1.27 1.27)) (justify left) hide)
     )
@@
       (effects (font (size 1.27 1.27)) (justify left))
     )
-    (property "Value" "R_Pack04_Split" (at 184.15 36.83 0)
+    (property "Value" "4x100" (at 184.15 36.83 0)
       (effects (font (size 1.27 1.27)) (justify left) hide)
     )
@@
       (effects (font (size 1.27 1.27)) (justify left))
     )
-    (property "Value" "R_Pack04_Split" (at 180.34 36.83 0)
+    (property "Value" "4x100" (at 180.34 36.83 0)
       (effects (font (size 1.27 1.27)) (justify left) hide)
     )

Commit message: MRES diode fix, use more common BGKR LED pinout and larger footprint.
Parts:
- renumbered C2 to C11, C8 to C12, C8 to C14, C912 to C29, C912 to C30, C1 to C32, C1 to C46, C1 to C47, C1 to C48, C1 to C49, C1 to C50, C1 to C51, C1 to C9, FB7 to FB13, R3 to R10, R3 to R11, R3 to R12, R3 to R14, R3 to R15
