File: 32X_main2.kicad_sch (KiCad schematic)
At the start: 54 parts, among them IC501 SH2 M, IC502 SH2 S, IC503 µPD4502161, IC504 315-5818, IC506 315-5781, IC507 TC511664, IC508 TC511664, IC509 74AC04, IC510 RHSRL33A

Commit message: Various fixes for r1.4 release.
Changed lines of the file:
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@@
 (kicad_sch
-	(version 20231120)
+	(version 20250114)
 	(generator "eeschema")
-	(generator_version "8.0")
+	(generator_version "9.0")
 	(paper "A3")
 	(title_block
 		(title "32X Main 2")
-		(date "2023-11-29")
-		(rev "1.3")
+		(date "2025-06-05")
+		(rev "1.4")
 		(company "By Cosam")
 		(comment 1 "Neptune")
 	)
+	(rectangle
+		(start 15.875 257.175)
+		(end 109.22 283.21)
+		(stroke
+			(width 0)
+			(type dash)
+		)
+		(fill
+			(type none)
+		)
+	)
+	(text "315-0922\n315-0922A\n315-0998"
+		(exclude_from_sim no)
+		(at 57.15 273.05 0)
+		(effects
+			(font
+				(size 1.27 1.27)
+			)
+			(justify left bottom)
+		)
+	)
+	(text "* Incorrectly labeled 14\n  on original 32X schematic"
+		(exclude_from_sim no)
+		(at 269.24 282.575 0)
+		(effects
+			(font
+				(size 1.27 1.27)
+			)
+			(justify left bottom)
+		)
+	)
+	(text "VA1 ONLY"
+		(exclude_from_sim no)
+		(at 59.69 262.255 0)
+		(effects
+			(font
+				(size 2.54 2.54)
+			)
+			(justify left bottom)
+		)
+	)
+	(text "*"
+		(exclude_from_sim no)
+		(at 296.545 78.105 0)
+		(effects
+			(font
+				(size 1.27 1.27)
+			)
+			(justify left bottom)
+		)
+	)
+	(text "IC502 Part No."
+		(exclude_from_sim no)
+		(at 57.15 266.7 0)
+		(effects
+			(font
+				(size 1.27 1.27)
+				(bold yes)
+			)
+			(justify left bottom)
+		)
+	)
+	(text "Value"
+		(exclude_from_sim no)
+		(at 95.885 266.7 0)
+		(effects
+			(font
+				(size 1.27 1.27)
+				(thickness 0.254)
+				(bold yes)
+			)
+			(justify left bottom)
+		)
+	)
+	(text "Description"
+		(exclude_from_sim no)
+		(at 74.93 266.7 0)
+		(effects
+			(font
+				(size 1.27 1.27)
+				(bold yes)
+			)
+			(justify left bottom)
+		)
+	)
+	(text "47pF\n100pF\n100pF"
+		(exclude_from_sim no)
+		(at 95.885 273.05 0)
+		(effects
+			(font
+				(size 1.27 1.27)
+			)
+			(justify left bottom)
+		)
+	)
+	(text "Extra decoupling for SH-2"
+		(exclude_from_sim no)
+		(at 365.125 114.935 0)
+		(effects
+			(font
+				(size 1.27 1.27)
+			)
+			(justify left bottom)
+		)
+	)
+	(text "Originally C96 and C97, which are THT capacitors\nsoldered directly to the chips on VA1 main boards.\nRenumbered 6xx to replace with SMD parts."
+		(exclude_from_sim no)
+		(at 57.15 280.67 0)
+		(effects
+			(font
+				(size 1.27 1.27)
+			)
+			(justify left bottom)
+		)
+	)
+	(text "HD6417095/F23\nHD6417095/F28\nHD6417095/F28"
+		(exclude_from_sim no)
+		(at 74.93 273.05 0)
+		(effects
+			(font
+				(size 1.27 1.27)
+			)
+			(justify left bottom)
+		)
+	)
+	(text "*"
+		(exclude_from_sim no)
+		(at 296.545 172.72 0)
+		(effects
+			(font
+				(size 1.27 1.27)
+			)
+			(justify left bottom)
+		)
+	)
 	(junction
 		(at 236.855 88.265)
@@
 		)
 	)
-	(rectangle
-		(start 15.875 257.175)
-		(end 109.22 283.21)
-		(stroke
-			(width 0)
-			(type dash)
-		)
-		(fill
-			(type none)
-		)
-	)
-	(text "315-0922\n315-0922A\n315-0998"
-		(exclude_from_sim no)
-		(at 57.15 273.05 0)
-		(effects
-			(font
-				(size 1.27 1.27)
-			)
-			(justify left bottom)
-		)
-	)
-	(text "* Incorrectly labeled 14\n  on original 32X schematic"
-		(exclude_from_sim no)
-		(at 269.24 282.575 0)
-		(effects
-			(font
-				(size 1.27 1.27)
-			)
-			(justify left bottom)
-		)
-	)
-	(text "VA1 ONLY"
-		(exclude_from_sim no)
-		(at 59.69 262.255 0)
-		(effects
-			(font
-				(size 2.54 2.54)
-			)
-			(justify left bottom)
-		)
-	)
-	(text "*"
-		(exclude_from_sim no)
-		(at 296.545 78.105 0)
-		(effects
-			(font
-				(size 1.27 1.27)
-			)
-			(justify left bottom)
-		)
-	)
-	(text "IC502 Part No."
-		(exclude_from_sim no)
-		(at 57.15 266.7 0)
-		(effects
-			(font
-				(size 1.27 1.27)
-				(bold yes)
-			)
-			(justify left bottom)
-		)
-	)
-	(text "Value"
-		(exclude_from_sim no)
-		(at 95.885 266.7 0)
-		(effects
-			(font
-				(size 1.27 1.27)
-				(thickness 0.254)
-				(bold yes)
-			)
-			(justify left bottom)
-		)
-	)
-	(text "Description"
-		(exclude_from_sim no)
-		(at 74.93 266.7 0)
-		(effects
-			(font
-				(size 1.27 1.27)
-				(bold yes)
-			)
-			(justify left bottom)
-		)
-	)
-	(text "47pF\n100pF\n100pF"
-		(exclude_from_sim no)
-		(at 95.885 273.05 0)
-		(effects
-			(font
-				(size 1.27 1.27)
-			)
-			(justify left bottom)
-		)
-	)
-	(text "Extra decoupling for SH-2"
-		(exclude_from_sim no)
-		(at 365.125 114.935 0)
-		(effects
-			(font
-				(size 1.27 1.27)
-			)
-			(justify left bottom)
-		)
-	)
-	(text "Originally C96 and C97, which are THT capacitors\nsoldered directly to the chips on VA1 main boards.\nRenumbered 6xx to replace with SMD parts."
-		(exclude_from_sim no)
-		(at 57.15 280.67 0)
-		(effects
-			(font
-				(size 1.27 1.27)
-			)
-			(justify left bottom)
-		)
-	)
-	(text "HD6417095/F23\nHD6417095/F28\nHD6417095/F28"
-		(exclude_from_sim no)
-		(at 74.93 273.05 0)
-		(effects
-			(font
-				(size 1.27 1.27)
-			)
-			(justify left bottom)
-		)
-	)
-	(text "*"
-		(exclude_from_sim no)
-		(at 296.545 172.72 0)
-		(effects
-			(font
-				(size 1.27 1.27)
-			)
-			(justify left bottom)
-		)
-	)
